File: High-density-proto-board.kicad_pcb (KiCad board)
At the start: 2 copper layers, 0 parts

Commit message: Mostly done.
Parts:
- added G***: OSHW-logo_silkscreen_5mm, oshw-logo:OSHW-logo_silkscreen_5mm, B.Cu at (112.4, 88.8)
- added G***: LED_smile_silkscreen_5mm, led-smile:LED_smile_silkscreen_5mm, B.Cu at (28.6, 88.8)
- added P?: VAL**, my_parts:MADW__SIL-1, F.Cu at (22.9, 66.0)
- added P?: VAL**, my_parts:MADW__SIL-8, F.Cu at (56.5, 77.5)
- added P?: VAL**, my_parts:MADW__SIL-8-1.27mm, F.Cu at (92.1, 101.6)
- added P?: VAL**, my_parts:MADW__SIL-8-1.27mm, F.Cu at (92.1, 99.1)
- added P?: VAL**, my_parts:MADW__SIL-8-1.27mm, F.Cu at (92.1, 96.5)
- added P?: VAL**, my_parts:MADW__SIL-8-1.27mm, F.Cu at (92.1, 94.0)
- added P?: VAL**, my_parts:MADW__SIL-8-1.27mm, F.Cu at (92.1, 83.8)
- added P?: VAL**, my_parts:MADW__SIL-8-1.27mm, F.Cu at (92.1, 81.3)
- added P?: VAL**, my_parts:MADW__SIL-8-1.27mm, F.Cu at (92.1, 78.7)
- added P?: VAL**, my_parts:MADW__SIL-8-1.27mm, F.Cu at (92.1, 76.2)
- added P?: VAL**, my_parts:MADW__SIL-8-1.27mm, F.Cu at (92.1, 73.7)
- added P?: VAL**, my_parts:MADW__SIL-8, F.Cu at (97.2, 95.2)
- added P?: VAL**, my_parts:MADW__SIL-8, F.Cu at (111.1, 82.5)
- added P?: VAL**, my_parts:MADW__SIL-8, F.Cu at (97.2, 100.3)
- added P?: VAL**, my_parts:MADW__SIL-8, F.Cu at (97.2, 102.9)
- added P?: VAL**, my_parts:MADW__SIL-8, F.Cu at (97.2, 92.7)
- added P?: VAL**, my_parts:MADW__SIL-8, F.Cu at (97.2, 82.5)
- added P?: VAL**, my_parts:MADW__SIL-8, F.Cu at (97.2, 77.5)
- added P?: VAL**, my_parts:MADW__SIL-8, F.Cu at (97.2, 74.9)
- added P?: VAL**, my_parts:MADW__SIL-8, F.Cu at (97.2, 85.1)
- added P?: VAL**, my_parts:MADW__SIL-8-1.27mm, F.Cu at (102.2, 73.7)
- added P?: VAL**, my_parts:MADW__SIL-8-1.27mm, F.Cu at (61.6, 73.7)
- added P?: VAL**, my_parts:MADW__SIL-8, F.Cu at (56.5, 85.1)
- added P?: VAL**, my_parts:MADW__SIL-8, F.Cu at (111.1, 80.0)
- added P?: VAL**, my_parts:MADW__SIL-8, F.Cu at (56.5, 74.9)
- added P?: VAL**, my_parts:MADW__SIL-8, F.Cu at (56.5, 80.0)
- added P?: VAL**, my_parts:MADW__SIL-8, F.Cu at (56.5, 82.5)
- added P?: VAL**, my_parts:MADW__SIL-8, F.Cu at (56.5, 92.7)
- added P?: VAL**, my_parts:MADW__SIL-8, F.Cu at (56.5, 102.9)
- added P?: VAL**, my_parts:MADW__SIL-8, F.Cu at (56.5, 100.3)
- added P?: VAL**, my_parts:MADW__SIL-8, F.Cu at (56.5, 97.8)
- added P?: VAL**, my_parts:MADW__SIL-8, F.Cu at (56.5, 95.2)
- added P?: VAL**, my_parts:MADW__SIL-8-1.27mm, F.Cu at (51.4, 73.7)
- added P?: VAL**, my_parts:MADW__SIL-8-1.27mm, F.Cu at (51.4, 76.2)
- added P?: VAL**, my_parts:MADW__SIL-8, F.Cu at (111.1, 77.5)
- added P?: VAL**, my_parts:MADW__SIL-8-1.27mm, F.Cu at (51.4, 78.7)
- added P?: VAL**, my_parts:MADW__SIL-8-1.27mm, F.Cu at (51.4, 81.3)
- added P?: VAL**, my_parts:MADW__SIL-8-1.27mm, F.Cu at (51.4, 83.8)
- added P?: VAL**, my_parts:MADW__SIL-8-1.27mm, F.Cu at (51.4, 94.0)
- added P?: VAL**, my_parts:MADW__SIL-8-1.27mm, F.Cu at (51.4, 96.5)
- added P?: VAL**, my_parts:MADW__SIL-8-1.27mm, F.Cu at (51.4, 99.1)
- added P?: VAL**, my_parts:MADW__SIL-8-1.27mm, F.Cu at (51.4, 101.6)
- added P?: VAL**, my_parts:MADW__SIL-8-1.27mm, F.Cu at (51.4, 104.1)
- added P?: VAL**, my_parts:MADW__SIL-8-1.27mm, F.Cu at (61.6, 76.2)
- added P?: VAL**, my_parts:MADW__SIL-8-1.27mm, F.Cu at (61.6, 78.7)
- added P?: VAL**, my_parts:MADW__SIL-8, F.Cu at (111.1, 74.9)
- added P?: VAL**, my_parts:MADW__SIL-8-1.27mm, F.Cu at (61.6, 81.3)
- added P?: VAL**, my_parts:MADW__SIL-8-1.27mm, F.Cu at (61.6, 83.8)
- added P?: VAL**, my_parts:MADW__SIL-8-1.27mm, F.Cu at (61.6, 104.1)
- added P?: VAL**, my_parts:MADW__SIL-8-1.27mm, F.Cu at (61.6, 101.6)
- added P?: VAL**, my_parts:MADW__SIL-8-1.27mm, F.Cu at (61.6, 99.1)
- added P?: VAL**, my_parts:MADW__SIL-8-1.27mm, F.Cu at (61.6, 96.5)
- added P?: VAL**, my_parts:MADW__SIL-8-1.27mm, F.Cu at (61.6, 94.0)
- added P?: VAL**, my_parts:MADW__SIL-8-1.27mm, F.Cu at (51.4, 106.7)
- added P?: VAL**, my_parts:MADW__SIL-8-1.27mm, F.Cu at (61.6, 106.7)
- added P?: VAL**, my_parts:MADW__SIL-8, F.Cu at (56.5, 108.0)
- added P?: VAL**, my_parts:MADW__SIL-8, F.Cu at (111.1, 69.8)
- added P?: VAL**, my_parts:MADW__SIL-8, F.Cu at (56.5, 110.5)
- added P?: VAL**, my_parts:MADW__SIL-8-1.27mm, F.Cu at (61.6, 111.8)
- added P?: VAL**, my_parts:MADW__SIL-8-1.27mm, F.Cu at (51.4, 111.8)
- added P?: VAL**, my_parts:MADW__SIL-8-1.27mm, F.Cu at (51.4, 71.1)
- added P?: VAL**, my_parts:MADW__SIL-8-1.27mm, F.Cu at (61.6, 71.1)
- added P?: VAL**, my_parts:MADW__SIL-8, F.Cu at (56.5, 69.8)
- added P?: VAL**, my_parts:MADW__SIL-8, F.Cu at (56.5, 67.3)
- added P?: VAL**, my_parts:MADW__SIL-8-1.27mm, F.Cu at (61.6, 66.0)
- added P?: VAL**, my_parts:MADW__SIL-8-1.27mm, F.Cu at (51.4, 66.0)
- added P?: VAL**, my_parts:MADW__SIL-8-1.27mm, F.Cu at (31.1, 66.0)
- added P?: VAL**, my_parts:MADW__SIL-8, F.Cu at (111.1, 67.3)
- added P?: VAL**, my_parts:MADW__SIL-8-1.27mm, F.Cu at (41.3, 66.0)
- added P?: VAL**, my_parts:MADW__SIL-8, F.Cu at (36.2, 67.3)
- added P?: VAL**, my_parts:MADW__SIL-8, F.Cu at (36.2, 69.8)
- added P?: VAL**, my_parts:MADW__SIL-8-1.27mm, F.Cu at (41.3, 71.1)
- added P?: VAL**, my_parts:MADW__SIL-8-1.27mm, F.Cu at (31.1, 71.1)
- added P?: VAL**, my_parts:MADW__SIL-8-1.27mm, F.Cu at (31.1, 111.8)
- added P?: VAL**, my_parts:MADW__SIL-8-1.27mm, F.Cu at (41.3, 111.8)
- added P?: VAL**, my_parts:MADW__SIL-8, F.Cu at (36.2, 110.5)
- added P?: VAL**, my_parts:MADW__SIL-8, F.Cu at (36.2, 108.0)
- added P?: VAL**, my_parts:MADW__SIL-8-1.27mm, F.Cu at (41.3, 106.7)
- added P?: VAL**, my_parts:MADW__SIL-8, F.Cu at (111.1, 85.1)
- added P?: VAL**, my_parts:MADW__SIL-8-1.27mm, F.Cu at (31.1, 106.7)
- added P?: VAL**, my_parts:MADW__SIL-8-1.27mm, F.Cu at (41.3, 94.0)
- added P?: VAL**, my_parts:MADW__SIL-8-1.27mm, F.Cu at (41.3, 96.5)
- added P?: VAL**, my_parts:MADW__SIL-8-1.27mm, F.Cu at (41.3, 99.1)
- added P?: VAL**, my_parts:MADW__SIL-8-1.27mm, F.Cu at (41.3, 101.6)
- added P?: VAL**, my_parts:MADW__SIL-8-1.27mm, F.Cu at (41.3, 104.1)
- added P?: VAL**, my_parts:MADW__SIL-8-1.27mm, F.Cu at (41.3, 83.8)
- added P?: VAL**, my_parts:MADW__SIL-8-1.27mm, F.Cu at (41.3, 81.3)
- added P?: VAL**, my_parts:MADW__SIL-8-1.27mm, F.Cu at (41.3, 78.7)
- added P?: VAL**, my_parts:MADW__SIL-8-1.27mm, F.Cu at (41.3, 76.2)
- added P?: VAL**, my_parts:MADW__SIL-8, F.Cu at (111.1, 102.9)
- added P?: VAL**, my_parts:MADW__SIL-8-1.27mm, F.Cu at (31.1, 104.1)
- added P?: VAL**, my_parts:MADW__SIL-8-1.27mm, F.Cu at (31.1, 101.6)
- added P?: VAL**, my_parts:MADW__SIL-8-1.27mm, F.Cu at (31.1, 99.1)
- added P?: VAL**, my_parts:MADW__SIL-8-1.27mm, F.Cu at (31.1, 96.5)
- added P?: VAL**, my_parts:MADW__SIL-8-1.27mm, F.Cu at (31.1, 94.0)
- added P?: VAL**, my_parts:MADW__SIL-8-1.27mm, F.Cu at (31.1, 83.8)
- added P?: VAL**, my_parts:MADW__SIL-8-1.27mm, F.Cu at (31.1, 81.3)
- added P?: VAL**, my_parts:MADW__SIL-8-1.27mm, F.Cu at (31.1, 78.7)
- added P?: VAL**, my_parts:MADW__SIL-8-1.27mm, F.Cu at (31.1, 76.2)
- added P?: VAL**, my_parts:MADW__SIL-8-1.27mm, F.Cu at (31.1, 73.7)
- added P?: VAL**, my_parts:MADW__SIL-8, F.Cu at (111.1, 100.3)
- added P?: VAL**, my_parts:MADW__SIL-8, F.Cu at (36.2, 95.2)
- added P?: VAL**, my_parts:MADW__SIL-8, F.Cu at (36.2, 97.8)
- added P?: VAL**, my_parts:MADW__SIL-8, F.Cu at (36.2, 100.3)
- added P?: VAL**, my_parts:MADW__SIL-8, F.Cu at (36.2, 92.7)
- added P?: VAL**, my_parts:MADW__SIL-8, F.Cu at (36.2, 82.5)
- added P?: VAL**, my_parts:MADW__SIL-8, F.Cu at (36.2, 80.0)
- added P?: VAL**, my_parts:MADW__SIL-8, F.Cu at (36.2, 77.5)
- added P?: VAL**, my_parts:MADW__SIL-8, F.Cu at (36.2, 74.9)
- added P?: VAL**, my_parts:MADW__SIL-8, F.Cu at (36.2, 85.1)
- added P?: VAL**, my_parts:MADW__SIL-8-1.27mm, F.Cu at (41.3, 73.7)
- added P?: VAL**, my_parts:MADW__SIL-1, F.Cu at (117.0, 88.9)
- added P?: VAL**, my_parts:MADW__SIL-8, F.Cu at (111.1, 97.8)
- added P?: VAL**, my_parts:MADW__SIL-8, F.Cu at (111.1, 95.2)
- added P?: VAL**, my_parts:MADW__SIL-8, F.Cu at (111.1, 92.7)
- added P?: VAL**, my_parts:MADW__SIL-8, F.Cu at (111.1, 110.5)
- added P?: VAL**, my_parts:MADW__SIL-8, F.Cu at (111.1, 108.0)
- added P?: VAL**, my_parts:MADW__SIL-8-1.27mm, F.Cu at (112.4, 66.0)
- added P?: VAL**, my_parts:MADW__SIL-8-1.27mm, F.Cu at (112.4, 71.1)
- added P?: VAL**, my_parts:MADW__SIL-8-1.27mm, F.Cu at (112.4, 73.7)
- added P?: VAL**, my_parts:MADW__SIL-8-1.27mm, F.Cu at (112.4, 76.2)
- added P?: VAL**, my_parts:MADW__SIL-8-1.27mm, F.Cu at (112.4, 78.7)
- added P?: VAL**, my_parts:MADW__SIL-1, F.Cu at (24.0, 88.9)
- added P?: VAL**, my_parts:MADW__SIL-8-1.27mm, F.Cu at (112.4, 81.3)
- added P?: VAL**, my_parts:MADW__SIL-8-1.27mm, F.Cu at (112.4, 83.8)
- added P?: VAL**, my_parts:MADW__SIL-8-1.27mm, F.Cu at (112.4, 111.8)
- added P?: VAL**, my_parts:MADW__SIL-8-1.27mm, F.Cu at (112.4, 106.7)
- added P?: VAL**, my_parts:MADW__SIL-8-1.27mm, F.Cu at (112.4, 104.1)
- added P?: VAL**, my_parts:MADW__SIL-8-1.27mm, F.Cu at (112.4, 101.6)
- added P?: VAL**, my_parts:MADW__SIL-8-1.27mm, F.Cu at (112.4, 99.1)
- added P?: VAL**, my_parts:MADW__SIL-8-1.27mm, F.Cu at (112.4, 96.5)
- added P?: VAL**, my_parts:MADW__SIL-8-1.27mm, F.Cu at (112.4, 94.0)
- added P?: VAL**, my_parts:MADW__SIL-8-1.27mm, F.Cu at (81.9, 73.7)
- added P?: VAL**, my_parts:MADW__SIL-8-1.27mm, F.Cu at (71.8, 81.3)
- added P?: VAL**, my_parts:MADW__SIL-8, F.Cu at (76.8, 85.1)
- added P?: VAL**, my_parts:MADW__SIL-8, F.Cu at (76.8, 74.9)
- added P?: VAL**, my_parts:MADW__SIL-8, F.Cu at (76.8, 80.0)
- added P?: VAL**, my_parts:MADW__SIL-8, F.Cu at (76.8, 82.5)
- added P?: VAL**, my_parts:MADW__SIL-8, F.Cu at (76.8, 92.7)
- added P?: VAL**, my_parts:MADW__SIL-8, F.Cu at (76.8, 102.9)
- added P?: VAL**, my_parts:MADW__SIL-8, F.Cu at (76.8, 100.3)
- added P?: VAL**, my_parts:MADW__SIL-8, F.Cu at (76.8, 95.2)
- added P?: VAL**, my_parts:MADW__SIL-8-1.27mm, F.Cu at (71.8, 73.7)
- added P?: VAL**, my_parts:MADW__SIL-8-1.27mm, F.Cu at (71.8, 76.2)
- added P?: VAL**, my_parts:MADW__SIL-8, F.Cu at (97.2, 97.8)
- added P?: VAL**, my_parts:MADW__SIL-8-1.27mm, F.Cu at (71.8, 78.7)
- added P?: VAL**, my_parts:MADW__SIL-8-1.27mm, F.Cu at (71.8, 83.8)
- added P?: VAL**, my_parts:MADW__SIL-8-1.27mm, F.Cu at (71.8, 94.0)
- added P?: VAL**, my_parts:MADW__SIL-8-1.27mm, F.Cu at (71.8, 96.5)
- added P?: VAL**, my_parts:MADW__SIL-8-1.27mm, F.Cu at (71.8, 99.1)
- added P?: VAL**, my_parts:MADW__SIL-8-1.27mm, F.Cu at (71.8, 101.6)
- added P?: VAL**, my_parts:MADW__SIL-8-1.27mm, F.Cu at (71.8, 104.1)
- added P?: VAL**, my_parts:MADW__SIL-8-1.27mm, F.Cu at (81.9, 76.2)
- added P?: VAL**, my_parts:MADW__SIL-8-1.27mm, F.Cu at (81.9, 78.7)
- added P?: VAL**, my_parts:MADW__SIL-8-1.27mm, F.Cu at (81.9, 81.3)
- added P?: VAL**, my_parts:MADW__SIL-8, F.Cu at (76.8, 97.8)
- added P?: VAL**, my_parts:MADW__SIL-8-1.27mm, F.Cu at (81.9, 83.8)
- added P?: VAL**, my_parts:MADW__SIL-8-1.27mm, F.Cu at (81.9, 104.1)
- added P?: VAL**, my_parts:MADW__SIL-8-1.27mm, F.Cu at (81.9, 101.6)
- added P?: VAL**, my_parts:MADW__SIL-8-1.27mm, F.Cu at (81.9, 99.1)
- added P?: VAL**, my_parts:MADW__SIL-8-1.27mm, F.Cu at (81.9, 96.5)
- added P?: VAL**, my_parts:MADW__SIL-8-1.27mm, F.Cu at (81.9, 94.0)
- added P?: VAL**, my_parts:MADW__SIL-8-1.27mm, F.Cu at (71.8, 106.7)
- added P?: VAL**, my_parts:MADW__SIL-8-1.27mm, F.Cu at (81.9, 106.7)
- added P?: VAL**, my_parts:MADW__SIL-8, F.Cu at (76.8, 108.0)
- added P?: VAL**, my_parts:MADW__SIL-8, F.Cu at (76.8, 110.5)
- added P?: VAL**, my_parts:MADW__SIL-8, F.Cu at (36.2, 102.9)
- added P?: VAL**, my_parts:MADW__SIL-8-1.27mm, F.Cu at (81.9, 111.8)
- added P?: VAL**, my_parts:MADW__SIL-8-1.27mm, F.Cu at (71.8, 111.8)
- added P?: VAL**, my_parts:MADW__SIL-8-1.27mm, F.Cu at (71.8, 71.1)
- added P?: VAL**, my_parts:MADW__SIL-8-1.27mm, F.Cu at (81.9, 71.1)
- added P?: VAL**, my_parts:MADW__SIL-8, F.Cu at (76.8, 69.8)
- added P?: VAL**, my_parts:MADW__SIL-8, F.Cu at (76.8, 67.3)
- added P?: VAL**, my_parts:MADW__SIL-8-1.27mm, F.Cu at (81.9, 66.0)
- added P?: VAL**, my_parts:MADW__SIL-8-1.27mm, F.Cu at (71.8, 66.0)
- added P?: VAL**, my_parts:MADW__SIL-8-1.27mm, F.Cu at (92.1, 66.0)
- added P?: VAL**, my_parts:MADW__SIL-8-1.27mm, F.Cu at (102.2, 66.0)
- added P?: VAL**, my_parts:MADW__SIL-8, F.Cu at (97.2, 80.0)
- added P?: VAL**, my_parts:MADW__SIL-8, F.Cu at (97.2, 67.3)
- added P?: VAL**, my_parts:MADW__SIL-8, F.Cu at (97.2, 69.8)
- added P?: VAL**, my_parts:MADW__SIL-8-1.27mm, F.Cu at (102.2, 71.1)
- added P?: VAL**, my_parts:MADW__SIL-8-1.27mm, F.Cu at (92.1, 71.1)
- added P?: VAL**, my_parts:MADW__SIL-8-1.27mm, F.Cu at (92.1, 111.8)
- added P?: VAL**, my_parts:MADW__SIL-8-1.27mm, F.Cu at (102.2, 111.8)
- added P?: VAL**, my_parts:MADW__SIL-8, F.Cu at (97.2, 110.5)
- added P?: VAL**, my_parts:MADW__SIL-8, F.Cu at (97.2, 108.0)
- added P?: VAL**, my_parts:MADW__SIL-8-1.27mm, F.Cu at (102.2, 106.7)
- added P?: VAL**, my_parts:MADW__SIL-8-1.27mm, F.Cu at (92.1, 106.7)
- added P?: VAL**, my_parts:MADW__SIL-8, F.Cu at (76.8, 77.5)
- added P?: VAL**, my_parts:MADW__SIL-8-1.27mm, F.Cu at (102.2, 94.0)
- added P?: VAL**, my_parts:MADW__SIL-8-1.27mm, F.Cu at (102.2, 96.5)
- added P?: VAL**, my_parts:MADW__SIL-8-1.27mm, F.Cu at (102.2, 99.1)
- added P?: VAL**, my_parts:MADW__SIL-8-1.27mm, F.Cu at (102.2, 101.6)
- added P?: VAL**, my_parts:MADW__SIL-8-1.27mm, F.Cu at (102.2, 104.1)
- added P?: VAL**, my_parts:MADW__SIL-8-1.27mm, F.Cu at (102.2, 83.8)
- added P?: VAL**, my_parts:MADW__SIL-8-1.27mm, F.Cu at (102.2, 81.3)
- added P?: VAL**, my_parts:MADW__SIL-8-1.27mm, F.Cu at (102.2, 78.7)
- added P?: VAL**, my_parts:MADW__SIL-8-1.27mm, F.Cu at (102.2, 76.2)
- added P?: VAL**, my_parts:MADW__SIL-8-1.27mm, F.Cu at (92.1, 104.1)
Routing:
- net (no net): track 0.00 -> 2011.7 mm
Other:
- board outline added: 99.1 x 49.5 mm
- net class Default: trace_width 0.2032 -> 0.4064
- board text added: "+"
- board text added: "-"
- board text added: "1"
- board text added: "10"
- board text added: "15"
- board text added: "20"
- board text added: "2014 - blog.spitzenpfeil.org V0.10.a"
- board text added: "25"
- board text added: "30"
- board text added: "35"
- board text added: "5"
- board text added: "A"
- board text added: "B"
- board text added: "C"
- board text added: "D"
- board text added: "E"
- board text added: "F"
- board text added: "G"
- board text added: "H"
- board text added: "I"
- board text added: "J"
