File: High-density-proto-board_50x50mm.kicad_pcb (KiCad board)
At the start: 2 copper layers, 48.3 x 49.5 mm, 89 parts

Commit message: Tweaks.
Parts:
- added G***: LOGO, LOGO, F.Cu at (45.1, 88.9)
- moved G*** 2.41 mm to (32.3, 88.9)
Other:
- board text added: "2014 - blog.spitzenpfeil.org 674 - V0.10.a"
- board text removed: "2014 - blog.spitzenpfeil.org V0.10.a"

Commit message: Oval pads. Good?
Parts:
- moved G*** 1.58 mm to (43.5, 89.0)
